Commit message: arm101实际和模拟(rviz)已经实现(tested),执行下面的启动文件 /home/kang/Documents/ros2_lekiwi/ignite.bash

File: src/lekiwi_vision/assets/so101_new_calib.urdf (robot description, URDF)
Before this commit: robot so101_new_calib, 8 links, 7 joints
Links:
- link base_link: geometry collision mesh filename=base_motor_holder_so101_v1.stl; collision mesh filename=base_so101_v2.stl
- link gripper_link: geometry collision mesh filename=sts3215_03a_v1.stl; collision mesh filename=wrist_roll_follower_so101_v1.stl
- link lower_arm_link: geometry collision mesh filename=motor_holder_so101_wrist_v1.stl; collision mesh filename=sts3215_03a_v1.stl
- link moving_jaw_so101_v1_link: geometry collision mesh filename=moving_jaw_so101_v1.stl; visual mesh filename=moving_jaw_so101_v1.stl
- link shoulder_link: geometry collision mesh filename=motor_holder_so101_base_v1.stl; collision mesh filename=rotation_pitch_so101_v1.stl
- link upper_arm_link: geometry collision mesh filename=sts3215_03a_v1.stl; collision mesh filename=upper_arm_so101_v1.stl
- link wrist_link: geometry collision mesh filename=sts3215_03a_no_horn_v1.stl; collision mesh filename=wrist_roll_pitch_so101_v2.stl
