Commit message: 原地夹球已经比较稳定，下一步准备加上底盘运动，实现远距离抓取

File: src/lekiwi_vision/urdf/lekiwi_robot.urdf.xacro (robot description, xacro)
@@ -1,65 +1,134 @@
 <?xml version="1.0"?>
-<!-- 定义机器人模型，名称为lekiwi_robot，引入xacro命名空间 -->
-<robot name="lekiwi_robot" xmlns:xacro="http://www.ros.org/wiki/xacro">
+<robot name="lekiwi_full_robot" xmlns:xacro="http://www.ros.org/wiki/xacro">
+    <!-- ========================================== -->
+    <!-- 0. 定义专属调色板，告别红屏报警 -->
+    <!-- ========================================== -->
+    <material name="LekiwiDarkGrey">
+        <color rgba="0.3 0.3 0.3 1.0"/>
+    </material>
+    <material name="LekiwiBlack">
+        <color rgba="0.1 0.1 0.1 1.0"/>
+    </material>
+    <material name="LekiwiWhite">
+        <color rgba="0.9 0.9 0.9 1.0"/>
+    </material>
+    <!-- 导入官方底盘 -->
+    <xacro:include filename="$(find lekiwi_vision)/urdf/LeKiwi.urdf" />
+    <link name="base_footprint"/>
+    <joint name="footprint_to_chassis" type="fixed">
+        <parent link="base_footprint"/>
+        <child link="base_plate_layer1-v5"/>
+        <origin xyz="0 0 0.05" rpy="0 0 0"/>
+    </joint>
     <!-- 引入lekiwi_vision包中的SO-101机械臂URDF模型 -->
     <xacro:include filename="$(find lekiwi_vision)/urdf/so101_arm.urdf" />
-    <!-- 定义底盘基准坐标系link（空link，用作整个模型的参考原点） -->
-    <link name="base_footprint">
-        </link>
     <!-- 定义机械臂与底盘之间的固定关节 -->
     <joint name="arm_to_base_joint" type="fixed">
-        <!-- 父link为底盘基准坐标系 -->
-        <parent link="base_footprint"/>
-        <!-- 子link为机械臂基座（对应so101_arm.urdf中的base_link） -->
+        <parent link="base_plate_layer2-v3"/>
         <child link="base_link"/>
-        <!-- 机械臂相对底盘的位置偏移：x方向前移0.1m，z方向上移0.05m -->
-        <origin xyz="0.1 0 0.05" rpy="0 0 0"/>
+        <origin xyz="0.00 0.04 0.007" rpy="0 0 1.57"/>
     </joint>
-    <!-- 定义支柱link，用于安装摄像头 -->
+    <link name="riser_base_link">
+        <visual>
+            <geometry>
+                <mesh filename="package://lekiwi_vision/meshes/riser_base.stl" scale="0.001 0.001 0.001"/>
+            </geometry>
+            <material name="LekiwiBlack"/> </visual>
+    </link>
+    <joint name="chassis_to_riser" type="fixed">
+        <parent link="base_plate_layer2-v3"/>
+        <child link="riser_base_link"/>
+        <origin xyz="-0.06 -0.037 0.007" rpy="0 0 0"/>
+    </joint>
     <link name="pillar_link">
-        <!-- 可视化属性 -->
         <visual>
-            <!-- 几何形状为长方体，尺寸为0.04m x 0.04m x 0.3m -->
             <geometry>
-                <box size="0.04 0.04 0.3"/> </geometry>
-            <!-- 材质为黄色 -->
-            <material name="yellow"><color rgba="1 1 0 1"/></material>
+                <mesh filename="package://lekiwi_vision/meshes/my_pillar.stl" scale="0.001 0.001 0.001"/>
+            </geometry>
+            <material name="LekiwiDarkGrey"/>
         </visual>
     </link>
-    <!-- 定义支柱与底盘之间的固定关节 -->
-    <joint name="pillar_to_base_joint" type="fixed">
-        <!-- 父link为底盘基准坐标系 -->
-        <parent link="base_footprint"/>
-        <!-- 子link为支柱 -->
+    <joint name="riser_to_pillar" type="fixed">
+        <parent link="riser_base_link"/>
         <child link="pillar_link"/>
-        <!-- 支柱相对底盘的位置偏移：x方向后移0.1m，z方向上移0.15m（支柱中心高度） -->
-        <origin xyz="-0.1 0 0.15" rpy="0 0 0"/>
+        <origin xyz="0.036 0.007 0.05" rpy="0 -1.57 0.5236"/>
     </joint>
-    <!-- 定义摄像头link（空link，用作摄像头安装点） -->
-    <link name="camera_link">
-        </link>
-    <!-- 定义摄像头俯仰关节，类型为旋转关节 -->
+    <!-- ========================================== -->
+    <!-- 2. 舵机固定件 (Servo Mount) -->
+    <!-- ========================================== -->
+    <link name="servo_mount_link">
+        <visual>
+            <geometry>
+                <mesh filename="package://lekiwi_vision/meshes/my_servo_mount.stl" scale="0.001 0.001 0.001"/>
+            </geometry>
+            <material name="LekiwiBlack"/>
+        </visual>
+    </link>
+    <joint name="pillar_to_mount" type="fixed">
+        <parent link="pillar_link"/>
+        <child link="servo_mount_link"/>
+        <origin xyz="0.25 0 0.025" rpy="0 1.57 0"/>
+    </joint>
+    <!-- ========================================== -->
+    <!-- 3. ST3215 舵机本体 (Servo Body) -->
+    <!-- ========================================== -->
+    <link name="st3215_servo_link">
+        <visual>
+            <geometry>
+                <mesh filename="package://lekiwi_vision/meshes/ST3215_Servo_Motor-v1.stl" scale="0.001 0.001 0.001"/>
+            </geometry>
+            <material name="LekiwiWhite"/>
+        </visual>
+    </link>
+    <joint name="mount_to_servo" type="fixed">
+        <parent link="servo_mount_link"/>
+        <child link="st3215_servo_link"/>
+        <origin xyz="-0.01 0.00 0.02" rpy="3.14 0 -1.57"/>
+    </joint>
+    <!-- ========================================== -->
+    <!-- 4. 相机固定件 (Camera Mount - 这是打在舵机上的塑料件) -->
+    <!-- ========================================== -->
+    <!-- 💥 修改点：名字从 camera_link 改成了 camera_mount_link -->
+    <link name="camera_mount_link">
+        <visual>
+            <origin xyz="0.0 0.0 -0.02" rpy="0 0 0"/>
+            <geometry>
+                <mesh filename="package://lekiwi_vision/meshes/my_camera_mount.stl" scale="0.001 0.001 0.001"/>
+            </geometry>
+            <material name="LekiwiBlack"/>
+        </visual>
+    </link>
+    <!-- 💥 核心云台关节：舵机带动【固定件】转动 -->
     <joint name="camera_pitch_joint" type="revolute">
-        <!-- 父link为支柱 -->
-        <parent link="pillar_link"/>
-        <!-- 子link为摄像头 -->
-        <child link="camera_link"/>
-        <!-- 摄像头相对支柱顶部的位置偏移：x方向前移0.02m，z方向上移0.15m -->
-        <origin xyz="0.02 0 0.15" rpy="0 0 0"/>
-        <!-- 旋转轴为Y轴（实现俯仰运动） -->
-        <axis xyz="0 1 0"/>
-        <!-- 关节限制：角度范围±0.785弧度（±45°），最大力矩10Nm，最大速度1rad/s -->
+        <parent link="st3215_servo_link"/>
+        <child link="camera_mount_link"/> <!-- 指向改名后的固定件 -->
+        <origin xyz="-0.025 -0.01 0.005" rpy="1.57 0 -1.57"/>
+        <axis xyz="1 0 0"/>
         <limit lower="-0.785" upper="0.785" effort="10" velocity="1"/>
     </joint>
-    <!-- 定义摄像头光学坐标系link（用于图像处理的坐标转换） -->
-    <link name="camera_color_optical_frame"/>
-    <!-- 定义摄像头光学坐标系与摄像头之间的固定关节 -->
-    <joint name="camera_optical_joint" type="fixed">
-        <!-- 父link为摄像头 -->
-        <parent link="camera_link"/>
-        <!-- 子link为光学坐标系 -->
-        <child link="camera_color_optical_frame"/>
-        <!-- 坐标变换：绕X轴旋转-90°，绕Z轴旋转-90°，将ROS坐标系转换为光学坐标系 -->
-        <origin xyz="0 0 0" rpy="-1.5708 0 -1.5708"/>
+    <!-- ========================================== -->
+    <!-- 5. RealSense 相机本体 (Camera Body) -->
+    <!-- ========================================== -->
+   <link name="camera_link">
+        <visual>
+            <origin xyz="0 -0.04 0" rpy="-1.57 0 -1.57"/>
+            <geometry>
+                <mesh filename="package://lekiwi_vision/meshes/d435.dae" />
+            </geometry>
+        </visual>
+        <collision>
+            <origin xyz="0 -0.04 0" rpy="-1.57 0 -1.57"/>
+            <geometry>
+                <box size="0.025 0.090 0.025"/>
+            </geometry>
+        </collision>
+    </link>
+    <!-- 💥 新增关节：用螺丝把【相机】锁死在【固定件】上！ -->
+    <joint name="mount_to_camera_joint" type="fixed">
+        <parent link="camera_mount_link"/> <!-- 爹是固定件 -->
+        <child link="camera_link"/>        <!-- 儿子是相机 -->
+        <!-- ⚠️ 亢哥注意：这里的 xyz 和 rpy 是相机相对于固定件螺丝孔的偏移量 -->
+        <!-- 你需要在 RViz 里微调这 6 个数字，让银色相机刚好贴合在你的黑色塑料支架上 -->
+        <origin xyz="-0.04 0 0.061" rpy="0 -1.57 1.57"/>
     </joint>
 </robot>

File: src/lekiwi_vision/urdf/so101_arm.urdf (robot description, URDF)
Before this commit: robot so101_new_calib, 8 links, 7 joints
Joints:
- joint elbow_flex: origin xyz=-0.11257 -0.028 1.73763e-16 rpy=-3.63608e-16 8.74301e-16 1.5708 -> xyz=-0.11257 -0.028 1.73763e-16 rpy=-3.63608e-16 8.74301e-16 1.1708
